Commit message: feat: ROS2/Gazebo/nav2 통합 레이어 개선 (Closes #154)
1. Nav2 YAML 중복 제거: 24개 controller YAML에서 공통 헤더
   (controller_server, progress_checker, goal_checker)를 base YAML로
   이동. 854줄 삭제, 플러그인별 override만 유지.
2. URDF 물리 강화: swerve steer joint type=revolute + <limit> 추가
   (effort=10Nm, velocity=3rad/s), damping 0.05→0.1
3. 센서 통합 확장: swerve_robot에 IMU (100Hz) + Depth Camera (15Hz,
   320x240) + PointCloud2 bridge 추가
4. E2E CI: ros2-ci.yml에 E2E 로직 테스트(22 tests) + 벤치마크 실행 추가
5. Dynamic Reconfigure: 기존 구현 확인 (lambda, Q/R, noise, CBF 등
   30+ 파라미터 런타임 변경 가능)

Co-Authored-By: Claude Opus 4.6 (1M context) <noreply@anthropic.com>

File: ros2_ws/src/mpc_controller_ros2/urdf/swerve_robot.urdf (robot description, URDF)
Before this commit: robot swerve_robot, 2 links, 1 joints
Links:
- added link camera_link, mass 0.05; collision box size=0.03 0.08 0.03; visual box size=0.03 0.08 0.03
- added link imu_link, mass 0.01; visual box size=0.02 0.02 0.01
Joints:
- added joint camera_joint: type fixed, parent base_link, child camera_link, origin xyz=0.25 0 ${base_height/2 + 0.08} rpy=0 0 0
- added joint imu_joint: type fixed, parent base_link, child imu_link, origin xyz=0 0 0.05 rpy=0 0 0
