Commit message: fix: anti-pitching + 후진 억제 — URDF 물리 강화 + lidar 상향 + MPPI 튜닝 (3/3 PASS)
URDF: mass 15→20kg, iyy 0.67(물리적 정확), CoM z=0.03(낮춤), lidar 0.35m+5°tilt, min_range 0.25m
Nav2: v_min -0.05, R_rate_v 3.0, prefer_forward 50.0, xy_goal_tolerance 0.50, obstacle_min_range 0.25

Co-Authored-By: Claude Opus 4.6 <noreply@anthropic.com>

File: ros2_ws/src/mpc_controller_ros2/urdf/differential_robot_ros2_control.urdf (robot description, URDF)
Before this commit: robot differential_robot, 5 links, 4 joints
Links:
- link base_link: mass 15.0 -> 20.0
Joints:
- joint lidar_joint: origin xyz=0.2 0 0.15 rpy=0 0 0 -> xyz=0.15 0 0.35 rpy=0 -0.087 0

Commit message: fix: Differential Drive URDF anti-pitching 개선 (Closes #147)
- 전방 캐스터 추가 → 3점(삼각형) → 4점(사각형) 접촉으로 피칭 억제
- 접촉 감쇠 kd: 100→500 (피칭 진동 억제 5배 강화)
- 구동휠 damping: 0.1→0.5 (반발 토크 댐핑 5배 강화)
- 기존 캐스터 rear_caster_wheel로 리네임 (명확성)

Co-Authored-By: Claude Opus 4.6 <noreply@anthropic.com>

File: ros2_ws/src/mpc_controller_ros2/urdf/differential_robot_ros2_control.urdf (robot description, URDF)
Before this commit: robot differential_robot, 5 links, 4 joints
Links:
- removed link caster_wheel
- added link front_caster_wheel, mass 1.0; collision sphere radius=0.05; visual sphere radius=0.05
- added link rear_caster_wheel, mass 1.0; collision sphere radius=0.05; visual sphere radius=0.05
Joints:
- removed joint caster_wheel_joint
- added joint front_caster_wheel_joint: type fixed, parent base_link, child front_caster_wheel, origin xyz=0.25 0 -0.05 rpy=0 0 0
- added joint rear_caster_wheel_joint: type fixed, parent base_link, child rear_caster_wheel, origin xyz=-0.25 0 -0.05 rpy=0 0 0

Commit message: fix: narrow_passage 장벽 위치 + 좀비 프로세스 정리 + DD lidar 바닥 검출 수정
- narrow_passage_world: 장벽 y=4,0,-4 → y=5,-2,-5 (스폰 위치 충돌 회피)
- launch: trap "" TERM + OnProcessExit/OnShutdown 종료 체인 추가
- cleanup_launch.sh: 좀비 프로세스 수동 정리 스크립트
- DD URDF lidar: pitch=-0.087rad 제거 (후방 바닥 검출 방지), 높이 0.35→0.20m

Co-Authored-By: Claude Opus 4.6 (1M context) <noreply@anthropic.com>

File: ros2_ws/src/mpc_controller_ros2/urdf/differential_robot_ros2_control.urdf (robot description, URDF)
Before this commit: robot differential_robot, 6 links, 5 joints
Joints:
- joint lidar_joint: origin xyz=0.15 0 0.35 rpy=0 -0.087 0 -> xyz=0.15 0 0.20 rpy=0 0 0
